File: src/DUB_with_Tono(ver1.0).sch (EAGLE design)
At the start: 3 parts

Commit message: ベタの追加
Parts:
- renumbered EDGE1 to DUB, U$2 to 遠野
Connections:
- removed net N$1: 遠野.P$1, 遠野.P$2, 遠野.P$3, 遠野.P$37, 遠野.P$38, 遠野.P$39, 遠野.P$4, 遠野.P$40
- net DIR_IN: now also 遠野.P$21
- net GND: now also 遠野.P$14, 遠野.P$15, 遠野.P$16, 遠野.P$17, 遠野.P$18, 遠野.P$23, 遠野.P$24, 遠野.P$25, 遠野.P$26, 遠野.P$27
- net GND_IN: now also 遠野.P$19
- net PWM_IN: now also 遠野.P$20
- net SA: now also 遠野.P$1, 遠野.P$2, 遠野.P$3, 遠野.P$37, 遠野.P$38, 遠野.P$39, 遠野.P$4, 遠野.P$40
- net SB: now also 遠野.P$33, 遠野.P$34, 遠野.P$35, 遠野.P$36, 遠野.P$5, 遠野.P$6, 遠野.P$7, 遠野.P$8
- net VCC: now also 遠野.P$10, 遠野.P$11, 遠野.P$12, 遠野.P$13, 遠野.P$28, 遠野.P$29, 遠野.P$30, 遠野.P$31, 遠野.P$32, 遠野.P$9
- net VCC_IN: now also 遠野.P$22
Other:
- note added: "5-5530843-4"
- note removed: "Tono logo"

Commit message: Eagle移行前_遠野ライブラリの修正
Changed lines of the file:
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@@
 <attribute name="VALUE" x="122.555" y="55.245" size="1.778" layer="96"/>
 </instance>
-<instance part="U$1" gate="G$1" x="101.6" y="12.7" smashed="yes"/>
+<instance part="U$1" gate="G$1" x="99.06" y="12.7" smashed="yes"/>
 </instances>
 <busses>
